File: pcb/qez.kicad_pcb (KiCad board)
At the start: 2 copper layers, 194.3 x 79 mm, 82 parts, among them U1 ATmega32U2-AU, U2 SRV05-4, X1 Crystal_GND24_Small

Commit message: moved switch
Parts:
- moved MX14 72.3 mm to (148.0, 155.6)
Other:
- net class Default removed
- net class Power removed
